File: LED_BOARD/grow-light-LEDS.kicad_pcb (KiCad board)
At the start: 2 copper layers, 125 x 70 mm, 32 parts, among them J1 Conn_02x04_Odd_Even

Commit message: Release v1.0
Parts:
- added J2: Conn_01x04, My_Library:FLIPPED_PRPC004SBCN-M71RC, F.Cu at (197.3, 134.8)
- J1: value Conn_02x04_Odd_Even -> Conn_01x04; footprint Connector_PinHeader_2.54mm:PinHeader_2x04_P2.54mm_Vertical_SMD -> My_Library:FLIPPED_PRPC004SBCN-M71RC
- moved REF** 21.0 mm to (157.3, 150.0)
- moved REF** 11.0 mm to (201.3, 106.0)
- moved J1 7.21 mm to (197.3, 121.3), turned to 180 degrees
- moved D1 0.50 mm to (169.2, 97.0)
- moved D10 0.50 mm to (89.2, 112.0)
- moved D11 0.50 mm to (169.2, 127.0)
- moved D12 0.50 mm to (149.2, 127.0)
- moved D13 0.50 mm to (128.6, 127.0)
- moved D14 0.50 mm to (109.2, 127.0)
- moved D15 0.50 mm to (89.2, 127.0)
- moved D16 0.50 mm to (169.2, 142.0)
- moved D17 0.50 mm to (149.2, 142.0)
- moved D18 0.50 mm to (128.6, 142.0)
- moved D19 0.50 mm to (109.2, 142.0)
- moved D2 0.50 mm to (149.2, 97.0)
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Connections:
- D1 pad 2: /1+ -> /4+
- D10 pad 1: /2- -> /3-
- D11 pad 2: /3+ -> /2+
- D15 pad 1: /3- -> /2-
- D16 pad 2: /4+ -> /1+
- D20 pad 1: /4- -> /1-
- D4 pad 1: /1- -> /4-
- D6 pad 2: /2+ -> /3+
- J1 pad 1: /2+ -> /4+
- J1 pad 2: /1+ -> /4-
- J1 pad 3: /2- -> /3+
- J1 pad 4: /1- -> /3-
Routing:
- net /4+: track 34.7 -> 45.3 mm
- net /2+: track 29.5 -> 35.8 mm
- net /4-: track 118.6 -> 124.2 mm
- net /3+: track 26.5 -> 31.5 mm
- net /3-: track 113.6 -> 110.0 mm
- net /1+: track 44.4 -> 41.2 mm
- net /1-: track 125.4 -> 122.5 mm
- net /2-: track 113.6 -> 114.8 mm
Other:
- outline, holes or cut-outs redrawn
- board text added: "- + - +"
- board text added: "GeoffGrowLight LED V1.0"
