File: LED_BOARD/grow-light-LEDS.kicad_sch (KiCad schematic)
At the start: 21 parts, among them J1 Conn_02x04_Odd_Even

Commit message: Release v1.0
Parts:
- removed J1: Conn_02x04_Odd_Even, Connector_PinHeader_2.54mm:PinHeader_2x04_P2.54mm_Vertical_SMD, symbol Connector_Generic:Conn_02x04_Odd_Even
- added J1, J2: Conn_01x04, My_Library:FLIPPED_PRPC004SBCN-M71RC, symbol Connector_Generic:Conn_01x04
Connections:
- net 1+: now also D16.2 (A), J2.4 (Pin_4); no longer D1.2 (A)
- net 1-: now also D20.1 (K), J2.3 (Pin_3); no longer D4.1 (K)
- net 2+: now also D11.2 (A), J2.2 (Pin_2); no longer D6.2 (A)
- net 2-: now also D15.1 (K), J2.1 (Pin_1); no longer D10.1 (K)
- net 3+: now also D6.2 (A), J1.3 (Pin_3); no longer D11.2 (A)
- net 3-: now also D10.1 (K), J1.4 (Pin_4); no longer D15.1 (K)
- net 4+: now also D1.2 (A), J1.1 (Pin_1); no longer D16.2 (A)
- net 4-: now also D4.1 (K), J1.2 (Pin_2); no longer D20.1 (K)
