File: MAIN_BOARD/grow-light.kicad_pcb (KiCad board)
At the start: 4 copper layers, 50 x 50 mm, 68 parts, among them J1 Conn_02x04_Odd_Even, J2 Connector, USB-TYPE-C-16P, J3 PROG, J4 UART, Q1 AO3401A, U1 HUSB238_xxxDD, U11 TPS61165DRV, U12 TPS61165DRV, U2 STM8S003F3P6TR, U3 USBLC6-2SC6, U4 TPS61165DRV, U5 TPS61165DRV, U7 HT7533

Commit message: Update board designs and production outputs
Parts:
- removed R2: 49.9kΩ, PCM_JLCPCB:R_0805
- added R11: 49.9kΩ, PCM_JLCPCB:R_0603, F.Cu at (121.0, 62.5)
- J1: footprint Connector_IDC:IDC-Header_2x04_P2.54mm_Vertical -> Connector_PinHeader_2.54mm:PinHeader_2x04_P2.54mm_Vertical
Routing:
- net GND: vias 44 -> 43

Commit message: Release v1.0
Parts:
- removed D1, D2, D3, D4: B5819WS, PCM_JLCPCB:D_SOD-323
- removed REF** (x4): MountingHole_2.2mm_M2_Pad_Via, MountingHole:MountingHole_2.2mm_M2_Pad_Via
- added D10: B16WS, PCM_JLCPCB:D_SOD-323, F.Cu at (138.5, 86.0)
- added D11: B16WS, PCM_JLCPCB:D_SOD-323, F.Cu at (138.5, 50.0)
- added D12: B16WS, PCM_JLCPCB:D_SOD-323, F.Cu at (138.5, 62.0)
- added D7: B16WS, PCM_JLCPCB:D_SOD-323, F.Cu at (138.5, 74.0)
- added H1: MountingHole_Pad, MountingHole:MountingHole_2.2mm_M2_Pad_Via, F.Cu at (155.0, 50.0)
- added H2: MountingHole_Pad, MountingHole:MountingHole_2.2mm_M2_Pad_Via, F.Cu at (155.0, 94.0)
- added H3: MountingHole_Pad, MountingHole:MountingHole_2.2mm_M2_Pad_Via, F.Cu at (111.0, 94.0)
- added H4: MountingHole_Pad, MountingHole:MountingHole_2.2mm_M2_Pad_Via, F.Cu at (111.0, 50.0)
- added TP_3v3: TestPoint, Connector_PinHeader_1.00mm:PinHeader_1x01_P1.00mm_Vertical, F.Cu at (127.5, 72.5)
- added TP_GND1: TestPoint, Connector_PinHeader_1.00mm:PinHeader_1x01_P1.00mm_Vertical, F.Cu at (156.0, 66.5)
- added TP_PWM1: TestPoint, Connector_PinHeader_1.00mm:PinHeader_1x01_P1.00mm_Vertical, F.Cu at (133.0, 93.0)
- added TP_VBUS1: TestPoint, Connector_PinHeader_1.00mm:PinHeader_1x01_P1.00mm_Vertical, F.Cu at (117.5, 66.5)
- added TP_Vin1: TestPoint, Connector_PinHeader_1.00mm:PinHeader_1x01_P1.00mm_Vertical, F.Cu at (130.5, 53.5)
- moved U3 13.8 mm to (149.5, 50.0)
- moved D6 6.26 mm to (117.5, 88.0)
- moved S1 6.26 mm to (117.5, 93.5)
- moved R17 6.21 mm to (114.9, 88.0)
- moved S2 5.83 mm to (126.5, 93.5)
- moved J1 5.82 mm to (147.2, 73.3), turned to 90 degrees
- moved C1 4.24 mm to (121.2, 53.8)
- moved C10 4.24 mm to (140.2, 50.2)
- moved C16 4.24 mm to (121.5, 85.2)
- moved C17 4.24 mm to (118.4, 82.5)
- moved C18 4.24 mm to (118.4, 79.6)
- moved C19 4.24 mm to (141.4, 76.2)
- moved C2 4.24 mm to (139.2, 79.5)
- moved C20 4.24 mm to (141.4, 88.2)
- moved C21 4.24 mm to (141.4, 52.2)
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Connections:
- C10 pad 1: /3+ -> /1+
- C11 pad 1: /4+ -> /2+
- C8 pad 1: /1+ -> /3+
- C9 pad 1: /2+ -> /4+
- J1 pad 1: /2+ -> /3-
- J1 pad 2: /1+ -> /2-
- J1 pad 3: /2- -> /3+
- J1 pad 4: /1- -> /2+
- J1 pad 5: /3- -> /4-
- J1 pad 6: /4- -> /1-
- J1 pad 7: /3+ -> /4+
- J1 pad 8: /4+ -> /1+
- R4 pad 1: /1- -> /3-
- R5 pad 1: /2- -> /4-
- R6 pad 1: /3- -> /1-
- R7 pad 1: /4- -> /2-
- U11 pad 1: /3- -> /1-
- U12 pad 1: /4- -> /2-
- U4 pad 1: /1- -> /3-
- U5 pad 1: /2- -> /4-
Routing:
- net /1+: track 10.2 -> 29.5 mm
- net /2-: track 25.3 -> 6.67 mm
- net /3-: track 25.7 -> 8.62 mm, vias 0 -> 1
- net /3+: track 26.4 -> 11.6 mm, vias 1 -> 0
- net /4-: track 8.94 -> 23.6 mm
- net /1-: track 10.5 -> 22.4 mm, vias 1 -> 0
- net /4+: track 13.6 -> 22.3 mm, vias 0 -> 1
- net Net-(U1-CC2): track 21.7 -> 30.2 mm
- net /PC6/PWM: track 58.1 -> 64.3 mm
- net Net-(U1-D+): track 35.1 -> 30.4 mm
- net Net-(U1-CC1): track 23.8 -> 28.4 mm
- net GND: track 10.2 -> 6.08 mm, vias 43 -> 46
- net Net-(U1-D-): track 35.0 -> 31.1 mm
- net /2+: track 18.5 -> 16.0 mm
- net VBUS: track 4.49 -> 6.99 mm
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- added copper zone on In1.Cu, net /USB_VBUS
- added copper zone on In2.Cu, net /USB_VBUS
Other:
- outline, holes or cut-outs redrawn
- board text added: "- + - +"
- board text added: "20W PD"
- board text added: "3v3"
- board text added: "GND"
- board text added: "Geoff Grow Light V1.0"
- board text added: "NRST"
- board text added: "RX"
- board text added: "SWIM"
- board text added: "TX"
