File: MAIN_BOARD/grow-light.kicad_sch (KiCad schematic)
At the start: 36 parts, among them J1 Conn_02x04_Odd_Even, J2 Connector, USB-TYPE-C-16P, J3 PROG, J4 UART, Q1 AO3401A, U1 HUSB238_xxxDD, U2 STM8S003F3P6TR, U3 USBLC6-2SC6, U7 HT7533

Commit message: Update board designs and production outputs
Parts:
- J1: footprint Connector_IDC:IDC-Header_2x04_P2.54mm_Vertical -> Connector_PinHeader_2.54mm:PinHeader_2x04_P2.54mm_Vertical
Changed lines of the file:
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@@
 			)
 		)
-		(property "Footprint" "Connector_IDC:IDC-Header_2x04_P2.54mm_Vertical"
+		(property "Footprint" "Connector_PinHeader_2.54mm:PinHeader_2x04_P2.54mm_Vertical"
 			(at 231.14 27.94 0)
 			(hide yes)

Commit message: Release v1.0
Parts:
- added H1, H2, H3, H4: MountingHole_Pad, MountingHole:MountingHole_2.2mm_M2_Pad_Via, symbol Mechanical:MountingHole_Pad
- added TP_3v3, TP_GND1, TP_PWM1, TP_VBUS1, TP_Vin1: TestPoint, Connector_PinHeader_1.00mm:PinHeader_1x01_P1.00mm_Vertical, symbol Connector:TestPoint
- J1: KiLib_Generator (none) -> connector/pin_header_socket
- U1: LCSC (none) -> C7471904
- U3: LCSC C7471904 -> C7519
Connections:
- net +3.3V: now also TP_3v3.1
- net 1+: now also J1.8 (Pin_8); no longer J1.2 (Pin_2)
- net 1-: now also J1.6 (Pin_6); no longer J1.4 (Pin_4)
- net 2+: now also J1.4 (Pin_4); no longer J1.1 (Pin_1)
- net 2-: now also J1.2 (Pin_2); no longer J1.3 (Pin_3)
- net 3+: now also J1.3 (Pin_3); no longer J1.7 (Pin_7)
- net 3-: now also J1.1 (Pin_1); no longer J1.5 (Pin_5)
- net 4+: now also J1.7 (Pin_7); no longer J1.8 (Pin_8)
- net 4-: now also J1.5 (Pin_5); no longer J1.6 (Pin_6)
- net GND: now also TP_GND1.1
- net LED_driver1/Vin: now also TP_Vin1.1
- net PC6/PWM: now also TP_PWM1.1
- net VBUS: now also TP_VBUS1.1
- no-connect marks 13 -> 17
