File: MAIN_BOARD/led_driver.kicad_sch (KiCad schematic)
At the start: 7 parts, among them U4 TPS61165DRV

Commit message: Release v1.0
Parts:
- removed D1: B5819WS, PCM_JLCPCB:D_SOD-323, symbol PCM_JLCPCB-Diodes:Schottky,B5819WS,(2)
- added D7: B16WS, PCM_JLCPCB:D_SOD-323, symbol PCM_JLCPCB-Diodes:Schottky,B16WS
- L1: KiLib_Generator (none) -> inductor/SMD
- U4: LCSC (none) -> C122568
Connections:
- net LED+: now also D7.1
- net at L1.2, U4.4 (SW): now also D7.2
